Commit message: fix link names

File: jackal_description/urdf/accessories/lidar/OS1-32.urdf.xacro (robot description, xacro)
@@ -6,5 +6,5 @@
       imu_link:=os_imu
       lasers:=32
-      lidar_link:=lidar_link
+      lidar_link:=os_lidar
       min_angle:=-${M_PI}
       max_angle:=${M_PI}

File: jackal_description/urdf/gz/jackal.gazebo.xacro (robot description, xacro)
@@ -11,12 +11,12 @@
     <!-- Sensors plugin -->
     <!-- Imu sensor -->
-    <gazebo reference="${prefix}imu_link">
+    <gazebo reference="${prefix}imu_0_link">
       <gravity>true</gravity>
-      <sensor name="${prefix}imu_sensor" type="imu">
+      <sensor name="${prefix}imu_0_sensor" type="imu">
           <always_on>true</always_on>
           <update_rate>50</update_rate>
           <visualize>true</visualize>
-          <topic>${prefix}imu</topic>
-          <gz_frame_id>${prefix}imu_link</gz_frame_id>
+          <topic>${prefix}imu_0</topic>
+          <gz_frame_id>${prefix}imu_0_link</gz_frame_id>
           <imu>
               <noise>
@@ -40,12 +40,12 @@
     <!-- Realsense D435 -->
     <xacro:if value="${use_camera}">
-      <gazebo reference="${prefix}camera_link">
-        <sensor name="${prefix}rgbd_camera" type="rgbd_camera">
+      <gazebo reference="${prefix}camera_0_link">
+        <sensor name="${prefix}camera_0" type="rgbd_camera">
           <always_on>true</always_on>
           <update_rate>5.0</update_rate>
           <visualize>true</visualize>
-          <gz_frame_id>${prefix}camera_link</gz_frame_id>
+          <gz_frame_id>${prefix}camera_0_link</gz_frame_id>
           <!-- if gz_frame_id = ${prefix}camera_depth_optical_frame, rtabmap works -->
-          <topic>${prefix}rgbd_camera</topic>
+          <topic>${prefix}camera_0</topic>
           <camera>
             <horizontal_fov>1.3962634</horizontal_fov>

File: jackal_description/urdf/jackal_macro.urdf.xacro (robot description, xacro)
@@ -98,5 +98,5 @@
     </xacro:wheel>
     <!-- Default Internal IMU Link -->
-    <link name="${prefix}imu_link">
+    <link name="${prefix}imu_0_link">
       <inertial>
         <mass value="0.001" />
@@ -108,7 +108,7 @@
       </inertial>
     </link>
-    <joint name="${prefix}imu_joint" type="fixed">
-      <parent link="${prefix}chassis_link" />
-      <child link="${prefix}imu_link" />
+    <joint name="${prefix}imu_0_joint" type="fixed">
+      <parent link="${prefix}chassis_link" />
+      <child link="${prefix}imu_0_link" />
     </joint>
     <!-- Default NAVSAT Link -->
@@ -199,5 +199,5 @@
       <xacro:sensor_d435
           add_plug="${add_plug}"
-          name="camera"
+          name="camera_0"
           parent="mid_mount"
           prefix="${prefix}"
@@ -211,5 +211,4 @@
       <xacro:include filename="$(find jackal_description)/urdf/accessories/lidar/OS1-32.urdf.xacro" />
       <xacro:OS1-32
-          name="os"
           parent="mid_mount"
           prefix="${prefix}"
