Commit message: temporary fix lidar frame direction

File: jackal_description/urdf/jackal_macro.urdf.xacro (robot description, xacro)
@@ -214,5 +214,10 @@
           prefix="${prefix}"
           sim_gazebo="${sim_gazebo}">
-        <origin xyz="0.14685 0 0.02564" rpy="0 0 0" />
+        <xacro:if value="${sim_gazebo}">
+          <origin xyz="0.14685 0 0.02564" rpy="0 0 0" />
+        </xacro:if>
+        <xacro:unless value="${sim_gazebo}">
+          <origin xyz="0.14685 0 0.02564" rpy="0 0 ${M_PI}" />
+        </xacro:unless>
       </xacro:OS1-32>
     </xacro:if>
