Commit message: add arm ros2 controllers launch

File: jackal_description/urdf/macros.urdf.xacro (robot description, xacro)
@@ -51,4 +51,7 @@
       <xacro:insert_block name="origin" />
       <axis xyz="0 1 0" />
+      <!-- Test arms with rqt-joint-trajectory-controller pkg -->
+      <!-- <limit lower="-${M_PI}" upper="${M_PI}"
+              effort="1000.0" velocity="1000.0" /> -->
     </joint>
   </xacro:macro>
